File: m2b1/m2b1.sch (KiCad schematic (older format))
At the start: 57 parts, among them P3 MicroD-37Pins, P4 MicroD-37Pins, Q1 2N3227, Q10 2N3227, Q2 2N3227, Q3 2N3227, Q4 2N2222, Q5 2N3227, Q6 2N3227, Q7 2N3227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

Commit message: Eradicated net names taken from ME901-0666 -- the pinout was completely changed from early revs of that document.
Connections:
- net BUF_CHK renamed B18_SHFT
- net BUF_CHK_n renamed B18_SHFT_n
- net ENABLE_n renamed PGOOD_n
Changed lines of the file:
@@
 	1825 2150 1525 2150
 Text Label 900  2050 0    50   ~ 0
-ENABLE_n
+PGOOD_n
 Wire Wire Line
 	1825 2050 1400 2050
@@
 NONZERO
 Text Label 2725 1650 2    50   ~ 0
-BUF_CHK
+B18_SHFT
 Wire Wire Line
 	2325 1650 2725 1650
 Text Label 2775 2550 2    50   ~ 0
-BUF_CHK_n
+B18_SHFT_n
 Wire Wire Line
 	2325 2550 2775 2550
@@
 	5500 2650 5050 2650
 Text Label 5050 2650 0    50   ~ 0
-BUF_CHK
+B18_SHFT
 NoConn ~ 5500 2550
 NoConn ~ 5750 2900
@@
 	8300 3200 7950 3200
 Text Label 7950 3200 0    50   ~ 0
-ENABLE_n
+PGOOD_n
 Wire Wire Line
 	8650 2250 8950 2250
@@
 	5500 5250 5050 5250
 Text Label 5050 5250 0    50   ~ 0
-BUF_CHK_n
+B18_SHFT_n
 NoConn ~ 5500 5050
 NoConn ~ 5750 5400
@@
 	8300 5700 7950 5700
 Text Label 7950 5700 0    50   ~ 0
-ENABLE_n
+PGOOD_n
 Wire Wire Line
 	8650 4750 8950 4750

Commit message: Corrected a schematic error in module 3 board 1, which now makes much more sense. Also renamed the power good net to VFAIL.
Connections:
- net PGOOD_n renamed VFAIL
Changed lines of the file:
@@
 	1825 2150 1525 2150
 Text Label 900  2050 0    50   ~ 0
-PGOOD_n
+VFAIL
 Wire Wire Line
 	1825 2050 1400 2050
@@
 	8300 3200 7950 3200
 Text Label 7950 3200 0    50   ~ 0
-PGOOD_n
+VFAIL
 Wire Wire Line
 	8650 2250 8950 2250
@@
 	8300 5700 7950 5700
 Text Label 7950 5700 0    50   ~ 0
-PGOOD_n
+VFAIL
 Wire Wire Line
 	8650 4750 8950 4750

Commit message: Initial schematic for module 4, board 1, plus lots of associated net name updates. The shift register is done, but a lot of surrounding NOR logic still needs to be untangled.
Connections:
- net B18_SHFT renamed BUF16
- net B18_SHFT_n renamed BUF16_n
- net BITJ3P1 renamed B12SET
- net BITJ3P2 renamed B10SET
- net BITJ3P20 renamed B15SET
- net BITJ3P21 renamed B09SET
- net BITJ3P22 renamed B16SET
- net BITJ3P23 renamed B13SET
- net BITJ3P3 renamed B11SET
- net BITJ3P5 renamed B14SET
- net BITJ4P2 renamed B01SET
- net BITJ4P20 renamed B04SET
- net BITJ4P21 renamed B03SET
- net BITJ4P22 renamed B06SET
- net BITJ4P23 renamed B05SET
- net BITJ4P24 renamed B08SET
- net BITJ4P3 renamed B07SET
- net NONZERO renamed BUFSET
Changed lines of the file:
@@
 	1850 5500 1550 5500
 Text Label 1550 5500 0    50   ~ 0
-BITJ4P2
+B01SET
 Wire Wire Line
 	2350 5600 2700 5600
 Text Label 2700 5600 2    50   ~ 0
-BITJ4P20
+B04SET
 Wire Wire Line
 	2350 5500 2700 5500
 Text Label 2700 5500 2    50   ~ 0
-BITJ4P21
+B03SET
 Wire Wire Line
 	1850 5400 1550 5400
 Text Label 1550 5400 0    50   ~ 0
-BITJ4P3
+B07SET
 Wire Wire Line
 	2350 5400 2700 5400
 Text Label 2700 5400 2    50   ~ 0
-BITJ4P22
+B06SET
 Wire Wire Line
 	2350 5300 2700 5300
 Text Label 2700 5300 2    50   ~ 0
-BITJ4P23
+B05SET
 Wire Wire Line
 	2350 5200 2700 5200
 Text Label 2700 5200 2    50   ~ 0
-BITJ4P24
+B08SET
 Wire Wire Line
 	1825 3050 1525 3050
 Text Label 1525 3050 0    50   ~ 0
-BITJ3P2
+B10SET
 Wire Wire Line
 	1825 3150 1525 3150
 Text Label 1525 3150 0    50   ~ 0
-BITJ3P1
+B12SET
 Wire Wire Line
 	1825 2950 1525 2950
 Text Label 1525 2950 0    50   ~ 0
-BITJ3P3
+B11SET
 Wire Wire Line
 	1825 2750 1525 2750
 Text Label 1525 2750 0    50   ~ 0
-BITJ3P5
+B14SET
 Wire Wire Line
 	2325 3150 2675 3150
 Text Label 2675 3150 2    50   ~ 0
-BITJ3P20
+B15SET
 Wire Wire Line
 	2325 3050 2675 3050
 Text Label 2675 3050 2    50   ~ 0
-BITJ3P21
+B09SET
 Wire Wire Line
 	2325 2950 2675 2950
 Text Label 2675 2950 2    50   ~ 0
-BITJ3P22
+B16SET
 Wire Wire Line
 	2325 2850 2675 2850
 Text Label 2675 2850 2    50   ~ 0
-BITJ3P23
+B13SET
 Wire Wire Line
 	1850 5600 1550 5600
 Text Label 1550 5600 0    50   ~ 0
-NONZERO
+BUFSET
 Text Label 2725 1650 2    50   ~ 0
-B18_SHFT
+BUF16
 Wire Wire Line
 	2325 1650 2725 1650
 Text Label 2775 2550 2    50   ~ 0
-B18_SHFT_n
+BUF16_n
 Wire Wire Line
 	2325 2550 2775 2550
@@
 	4800 3400 5200 3400
 Text Label 5200 3400 2    50   ~ 0
-NONZERO
+BUFSET
 $Comp
 L gn_buffer:MC305 U4
@@
 	3700 4950 3300 4950
 Text Label 3300 4950 0    50   ~ 0
-BITJ4P21
+B03SET
 Wire Wire Line
 	3700 4850 3300 4850
 Text Label 3300 4850 0    50   ~ 0
-BITJ4P2
+B01SET
 Wire Wire Line
 	3700 4750 3300 4750
 Text Label 3300 4750 0    50   ~ 0
-BITJ4P20
+B04SET
 Wire Wire Line
 	3700 4650 3300 4650
 Text Label 3300 4650 0    50   ~ 0
-BITJ4P3
+B07SET
 Wire Wire Line
 	3700 4550 3300 4550
 Text Label 3300 4550 0    50   ~ 0
-BITJ4P22
+B06SET
 Wire Wire Line
 	3700 4450 3300 4450
 Text Label 3300 4450 0    50   ~ 0
-BITJ4P23
+B05SET
 Wire Wire Line
 	3700 4350 3300 4350
 Text Label 3300 4350 0    50   ~ 0
-BITJ4P24
+B08SET
 Wire Wire Line
 	3700 4250 3300 4250
 Text Label 3300 4250 0    50   ~ 0
-BITJ3P1
+B12SET
 Wire Wire Line
 	3700 4150 3300 4150
 Text Label 3300 4150 0    50   ~ 0
-BITJ3P21
+B09SET
 Wire Wire Line
 	3700 4050 3300 4050
 Text Label 3300 4050 0    50   ~ 0
-BITJ3P2
+B10SET
 Wire Wire Line
 	3700 3950 3300 3950
 Text Label 3300 3950 0    50   ~ 0
-BITJ3P22
+B16SET
 Wire Wire Line
 	3700 3850 3300 3850
 Text Label 3300 3850 0    50   ~ 0
-BITJ3P20
+B15SET
 Wire Wire Line
 	3700 3750 3300 3750
 Text Label 3300 3750 0    50   ~ 0
-BITJ3P3
+B11SET
 Wire Wire Line
 	3700 3650 3300 3650
 Text Label 3300 3650 0    50   ~ 0
-BITJ3P5
+B14SET
 Wire Wire Line
 	3700 3550 3300 3550
 Text Label 3300 3550 0    50   ~ 0
-BITJ3P23
+B13SET
 Text Notes 4200 2900 2    50   ~ 0
 Buffer Zero Detector
@@
 	5500 2650 5050 2650
 Text Label 5050 2650 0    50   ~ 0
-B18_SHFT
+BUF16
 NoConn ~ 5500 2550
 NoConn ~ 5750 2900
@@
 	5500 5250 5050 5250
 Text Label 5050 5250 0    50   ~ 0
-B18_SHFT_n
+BUF16_n
 NoConn ~ 5500 5050
 NoConn ~ 5750 5400

Commit message: Greatly cleaned up all of the schematics so far; everything passes DRC.
Parts:
- removed unit 2 of U1
- removed unit 2 of U2
- removed unit 2 of U3
- renumbered C3 to C1, C6 to C2, C1 to C3, C2 to C4, C4 to C5, C5 to C6
Other:
- note added: "Buffer Bit Set OR"
- note added: "Output Transformer Drivers"
- note removed: "Buffer Zero Detector"
- note removed: "Power Connections"
- note removed: "Transformer Drivers"
- moved on the sheet: C1, C2
